Commit message: endeffactor

File: arm_description/urdf/arm.xacro (robot description, xacro)
@@ -14,4 +14,10 @@
   <xacro:property name="l3_half" value="0.125"/>
   <xacro:property name="l4_half" value="0.10"/>
+    <!-- ===================== -->
+  <!-- MATERIALS -->
+  <!-- ===================== -->
+  <material name="wheel_black">
+    <color rgba="0.02 0.02 0.02 1.0"/>
+  </material>
   <!-- ===================== -->
   <!-- INERTIA MACRO -->
@@ -141,4 +147,30 @@
     <limit lower="-3.14" upper="3.14" effort="10" velocity="2.0"/>
   </joint>
+  <link name="tool0"/>
+    <joint name="wrist_to_tool0" type="fixed">
+      <parent link="arm_link_4"/>
+      <child link="tool0"/>
+      <!-- adjust xyz if needed -->
+      <origin xyz="0 0 ${l4}" rpy="0 0 0"/>
+    </joint>
+    <!-- ee_link : physical tool -->
+  <link name="ee_link">
+    <visual>
+      <geometry>
+        <box size="0.04 0.04 0.02"/>
+      </geometry>
+      <material name="wheel_black"/>
+    </visual>
+    <collision>
+      <geometry>
+        <box size="0.04 0.04 0.02"/>
+      </geometry>
+    </collision>
+  </link>
+    <joint name="tool0_to_ee" type="fixed">
+      <parent link="tool0"/>
+      <child link="ee_link"/>
+      <origin xyz="0.03 0 0"/>
+    </joint>
   <ros2_control name="ArmSystem" type="system">
     <hardware>

Commit message: arm_pos controller

File: arm_description/urdf/arm.xacro (robot description, xacro)
@@ -6,12 +6,14 @@
   <xacro:property name="r" value="0.03"/>
   <xacro:property name="m" value="2.0"/>
-  <xacro:property name="l1" value="0.20"/>
+  <xacro:property name="l1" value="0.10"/>
   <xacro:property name="l2" value="0.30"/>
   <xacro:property name="l3" value="0.25"/>
   <xacro:property name="l4" value="0.20"/>
-  <xacro:property name="l1_half" value="0.10"/>
+  <xacro:property name="l5" value="0.10"/>
+  <xacro:property name="l1_half" value="0.05"/>
   <xacro:property name="l2_half" value="0.15"/>
   <xacro:property name="l3_half" value="0.125"/>
   <xacro:property name="l4_half" value="0.10"/>
+  <xacro:property name="l5_half" value="0.05"/>
     <!-- ===================== -->
   <!-- MATERIALS -->
@@ -147,10 +149,47 @@
     <limit lower="-3.14" upper="3.14" effort="10" velocity="2.0"/>
   </joint>
+  <!-- ===================== -->
+  <!-- LINK 5 -->
+  <!-- ===================== -->
+  <!-- ===================== -->
+<!-- LINK 5 -->
+<!-- ===================== -->
+  <link name="arm_link_5">
+    <inertial>
+      <origin xyz="0 0 ${l5_half}"/>
+      <xacro:cyl_inertia m="1.0" r="0.025" l="${l5}"/>
+    </inertial>
+    <visual>
+      <origin xyz="0 0 ${l5_half}"/>
+      <geometry>
+        <cylinder length="${l5}" radius="0.025"/>
+      </geometry>
+    </visual>
+    <collision>
+      <origin xyz="0 0 ${l5_half}"/>
+      <geometry>
+        <cylinder length="${l5}" radius="0.025"/>
+      </geometry>
+    </collision>
+  </link>
+  <!-- Wrist roll joint (PERPENDICULAR) -->
+  <joint name="wrist_roll_joint" type="revolute">
+    <parent link="arm_link_4"/>
+    <child link="arm_link_5"/>
+    <!-- rotate joint frame by 90 deg -->
+    <origin xyz="0 0 ${l4}" rpy="1.5708 0 0"/>
+    <!-- rotation axis now perpendicular -->
+    <axis xyz="0 1 0"/>
+    <limit lower="-3.14" upper="3.14" effort="10" velocity="2.0"/>
+  </joint>
+    <!-- ===================== -->
+  <!-- END EFFECTOR -->
+  <!-- ===================== -->
   <link name="tool0"/>
     <joint name="wrist_to_tool0" type="fixed">
-      <parent link="arm_link_4"/>
+      <parent link="arm_link_5"/>
       <child link="tool0"/>
       <!-- adjust xyz if needed -->
-      <origin xyz="0 0 ${l4}" rpy="0 0 0"/>
+      <origin xyz="0 0 ${l5}" rpy="1.5708 0 0"/>
     </joint>
     <!-- ee_link : physical tool -->

Commit message: arm_pos controller

File: arm_description/urdf/arm.xacro (robot description, xacro)
@@ -237,4 +237,9 @@
       <state_interface name="velocity"/>
     </joint>
+    <joint name="wrist_roll_joint">
+      <command_interface name="position"/>
+      <state_interface name="position"/>
+      <state_interface name="velocity"/>
+    </joint>
     <joint name="FWRJ">
       <state_interface name="position"/>

Commit message: endeffactor for 2 joints

File: arm_description/urdf/arm.xacro (robot description, xacro)
@@ -124,5 +124,5 @@
   <!-- LINK 4 -->
   <!-- ===================== -->
-  <link name="arm_link_4">
+  <!-- <link name="arm_link_4">
     <inertial>
       <origin xyz="0 0 ${l4_half}"/>
@@ -141,6 +141,6 @@
       </geometry>
     </collision>
-  </link>
-  <joint name="wrist_joint" type="revolute">
+  </link> -->
+  <!-- <joint name="wrist_joint" type="revolute">
     <parent link="arm_link_3"/>
     <child link="arm_link_4"/>
@@ -148,12 +148,12 @@
     <axis xyz="0 1 0"/>
     <limit lower="-3.14" upper="3.14" effort="10" velocity="2.0"/>
-  </joint>
+  </joint> -->
   <!-- ===================== -->
   <!-- LINK 5 -->
   <!-- ===================== -->
   <!-- ===================== -->
-<!-- LINK 5 -->
-<!-- ===================== -->
-  <link name="arm_link_5">
+  <!-- LINK 5 -->
+  <!-- ===================== -->
+  <!-- <link name="arm_link_5">
     <inertial>
       <origin xyz="0 0 ${l5_half}"/>
@@ -172,15 +172,13 @@
       </geometry>
     </collision>
-  </link>
+  </link> -->
   <!-- Wrist roll joint (PERPENDICULAR) -->
-  <joint name="wrist_roll_joint" type="revolute">
+  <!-- <joint name="wrist_roll_joint" type="revolute">
     <parent link="arm_link_4"/>
     <child link="arm_link_5"/>
-    <!-- rotate joint frame by 90 deg -->
     <origin xyz="0 0 ${l4}" rpy="1.5708 0 0"/>
-    <!-- rotation axis now perpendicular -->
     <axis xyz="0 1 0"/>
     <limit lower="-3.14" upper="3.14" effort="10" velocity="2.0"/>
-  </joint>
+  </joint> -->
     <!-- ===================== -->
   <!-- END EFFECTOR -->
@@ -188,8 +186,8 @@
   <link name="tool0"/>
     <joint name="wrist_to_tool0" type="fixed">
-      <parent link="arm_link_5"/>
+      <parent link="arm_link_3"/>
       <child link="tool0"/>
       <!-- adjust xyz if needed -->
-      <origin xyz="0 0 ${l5}" rpy="1.5708 0 0"/>
+      <origin xyz="0 0 ${l3}" rpy="0 0 0"/>
     </joint>
     <!-- ee_link : physical tool -->
@@ -232,5 +230,5 @@
       <state_interface name="velocity"/>
     </joint>
-    <joint name="wrist_joint">
+    <!-- <joint name="wrist_joint">
       <command_interface name="position"/>
       <state_interface name="position"/>
@@ -241,5 +239,5 @@
       <state_interface name="position"/>
       <state_interface name="velocity"/>
-    </joint>
+    </joint> -->
     <joint name="FWRJ">
       <state_interface name="position"/>

Commit message: wrist_joint

File: arm_description/urdf/arm.xacro (robot description, xacro)
@@ -9,10 +9,10 @@
   <xacro:property name="l2" value="0.30"/>
   <xacro:property name="l3" value="0.25"/>
-  <xacro:property name="l4" value="0.20"/>
+  <xacro:property name="l4" value="0.10"/>
   <xacro:property name="l5" value="0.10"/>
   <xacro:property name="l1_half" value="0.05"/>
   <xacro:property name="l2_half" value="0.15"/>
   <xacro:property name="l3_half" value="0.125"/>
-  <xacro:property name="l4_half" value="0.10"/>
+  <xacro:property name="l4_half" value="0.05"/>
   <xacro:property name="l5_half" value="0.05"/>
     <!-- ===================== -->
@@ -124,5 +124,5 @@
   <!-- LINK 4 -->
   <!-- ===================== -->
-  <!-- <link name="arm_link_4">
+  <link name="arm_link_4">
     <inertial>
       <origin xyz="0 0 ${l4_half}"/>
@@ -141,6 +141,6 @@
       </geometry>
     </collision>
-  </link> -->
-  <!-- <joint name="wrist_joint" type="revolute">
+  </link>
+  <joint name="wrist_joint" type="revolute">
     <parent link="arm_link_3"/>
     <child link="arm_link_4"/>
@@ -148,5 +148,5 @@
     <axis xyz="0 1 0"/>
     <limit lower="-3.14" upper="3.14" effort="10" velocity="2.0"/>
-  </joint> -->
+  </joint>
   <!-- ===================== -->
   <!-- LINK 5 -->
@@ -186,8 +186,8 @@
   <link name="tool0"/>
     <joint name="wrist_to_tool0" type="fixed">
-      <parent link="arm_link_3"/>
+      <parent link="arm_link_4"/>
       <child link="tool0"/>
       <!-- adjust xyz if needed -->
-      <origin xyz="0 0 ${l3}" rpy="0 0 0"/>
+      <origin xyz="0 0 ${l4}" rpy="0 0 0"/>
     </joint>
     <!-- ee_link : physical tool -->
@@ -208,5 +208,5 @@
       <parent link="tool0"/>
       <child link="ee_link"/>
-      <origin xyz="0.03 0 0"/>
+      <origin xyz="0.0 0 0"/>
     </joint>
   <ros2_control name="ArmSystem" type="system">
@@ -230,10 +230,10 @@
       <state_interface name="velocity"/>
     </joint>
-    <!-- <joint name="wrist_joint">
-      <command_interface name="position"/>
-      <state_interface name="position"/>
-      <state_interface name="velocity"/>
-    </joint>
-    <joint name="wrist_roll_joint">
+    <joint name="wrist_joint">
+      <command_interface name="position"/>
+      <state_interface name="position"/>
+      <state_interface name="velocity"/>
+    </joint>
+    <!-- <joint name="wrist_roll_joint">
       <command_interface name="position"/>
       <state_interface name="position"/>

Commit message: gazebo simulation done for arm

File: arm_description/urdf/arm.xacro (robot description, xacro)
@@ -1,4 +1,5 @@
 <?xml version="1.0"?>
 <robot xmlns:xacro="http://www.ros.org/wiki/xacro">
+  <xacro:macro name="ebot_arm">
   <!-- ===================== -->
   <!-- PARAMETERS -->
@@ -211,8 +212,9 @@
     </joint>
   <ros2_control name="ArmSystem" type="system">
-    <hardware>
-      <!-- Fake hardware for simulation / RViz -->
-      <plugin>fake_components/GenericSystem</plugin>
-    </hardware>
+  <hardware>
+    <plugin>gz_ros2_control/GazeboSimSystem</plugin>
+    <!-- <plugin>mock_components/GenericSystem</plugin> -->
+    <param name="initial_positions">0 0 0 0</param>
+  </hardware>
     <joint name="base_rotation_joint">
       <command_interface name="position"/>
@@ -249,3 +251,4 @@
     </joint>
   </ros2_control>
+  </xacro:macro>
 </robot>

File: ebot_description/models/ebot/ebot_description.xacro (robot description, xacro)
@@ -1,6 +1,9 @@
 <?xml version="1.0"?>
 <robot name="ebot" xmlns:xacro="http://www.ros.org/wiki/xacro">
+  <xacro:arg name="use_gazebo" default="true"/>
   <xacro:include filename="$(find ebot_description)/models/ebot/ebot.gazebo" />
   <xacro:include filename="$(find arm_description)/urdf/arm.xacro" />
+  <xacro:include filename="$(find ebot_description)/models/ebot/ebot_gazebo_control.xacro"/>
+  <xacro:ebot_arm/>
   <!-- ===================== -->
   <!-- PROPERTIES -->
@@ -255,3 +258,4 @@
     <child link="imu_link"/>
   </joint>
+<xacro:ebot_gazebo_ros2_control/>
 </robot>

Commit message: ee_velocity control and arm integration

File: arm_description/urdf/arm.xacro (robot description, xacro)
@@ -10,10 +10,10 @@
   <xacro:property name="l2" value="0.30"/>
   <xacro:property name="l3" value="0.25"/>
-  <xacro:property name="l4" value="0.10"/>
+  <xacro:property name="l4" value="0.05"/>
   <xacro:property name="l5" value="0.10"/>
   <xacro:property name="l1_half" value="0.05"/>
   <xacro:property name="l2_half" value="0.15"/>
   <xacro:property name="l3_half" value="0.125"/>
-  <xacro:property name="l4_half" value="0.05"/>
+  <xacro:property name="l4_half" value="0.025"/>
   <xacro:property name="l5_half" value="0.05"/>
     <!-- ===================== -->
@@ -120,5 +120,5 @@
     <origin xyz="0 0 ${l2}"/>
     <axis xyz="0 1 0"/>
-    <limit lower="-1.57" upper="1.57" effort="15" velocity="1.5"/>
+    <limit lower="0.00" upper="3.1" effort="15" velocity="1.5"/>
   </joint>
   <!-- ===================== -->
@@ -213,6 +213,6 @@
   <ros2_control name="ArmSystem" type="system">
   <hardware>
-    <plugin>gz_ros2_control/GazeboSimSystem</plugin>
-    <!-- <plugin>mock_components/GenericSystem</plugin> -->
+    <!-- <plugin>gz_ros2_control/GazeboSimSystem</plugin> -->
+    <plugin>mock_components/GenericSystem</plugin>
     <param name="initial_positions">0 0 0 0</param>
   </hardware>
@@ -243,8 +243,10 @@
     </joint> -->
     <joint name="FWRJ">
+      <command_interface name="velocity"/>
       <state_interface name="position"/>
       <state_interface name="velocity"/>
     </joint>
     <joint name="FWLJ">
+      <command_interface name="velocity"/>
       <state_interface name="position"/>
       <state_interface name="velocity"/>

File: ebot_description/models/ebot/ebot_description.xacro (robot description, xacro)
@@ -68,5 +68,5 @@
     <parent link="ebot_base"/>
     <child link="arm_base_link"/>
-    <origin xyz="0 0 0.25" rpy="0 0 0"/>
+    <origin xyz="0 0 0.12" rpy="0 0 0"/>
   </joint>
   <!-- ===================== -->
@@ -128,4 +128,25 @@
   </joint>
   <!-- ===================== -->
+  <!-- TRANSMISSIONS -->
+  <!-- ===================== -->
+  <transmission name="FWR_trans">
+    <type>transmission_interface/SimpleTransmission</type>
+    <joint name="FWRJ">
+      <hardwareInterface>hardware_interface/VelocityJointInterface</hardwareInterface>
+    </joint>
+    <actuator name="FWR_motor">
+      <mechanicalReduction>1</mechanicalReduction>
+    </actuator>
+  </transmission>
+  <transmission name="FWL_trans">
+    <type>transmission_interface/SimpleTransmission</type>
+    <joint name="FWLJ">
+      <hardwareInterface>hardware_interface/VelocityJointInterface</hardwareInterface>
+    </joint>
+    <actuator name="FWL_motor">
+      <mechanicalReduction>1</mechanicalReduction>
+    </actuator>
+  </transmission>
+  <!-- ===================== -->
   <!-- OMNI CASTERS (SWIVEL + ROLL) -->
   <!-- ===================== -->

Commit message: build full arm

File: arm_description/urdf/arm.xacro (robot description, xacro)
@@ -1,4 +1,5 @@
 <?xml version="1.0"?>
 <robot xmlns:xacro="http://www.ros.org/wiki/xacro">
+<xacro:include filename="$(find arm_description)/urdf/simple_gripper.xacro"/>
   <xacro:macro name="ebot_arm">
   <!-- ===================== -->
@@ -11,10 +12,12 @@
   <xacro:property name="l3" value="0.25"/>
   <xacro:property name="l4" value="0.05"/>
-  <xacro:property name="l5" value="0.10"/>
+  <xacro:property name="l5" value="0.05"/>
+  <xacro:property name="l6" value="0.05"/>
   <xacro:property name="l1_half" value="0.05"/>
   <xacro:property name="l2_half" value="0.15"/>
   <xacro:property name="l3_half" value="0.125"/>
   <xacro:property name="l4_half" value="0.025"/>
-  <xacro:property name="l5_half" value="0.05"/>
+  <xacro:property name="l5_half" value="0.025"/>
+  <xacro:property name="l6_half" value="0.025"/>
     <!-- ===================== -->
   <!-- MATERIALS -->
@@ -22,4 +25,7 @@
   <material name="wheel_black">
     <color rgba="0.02 0.02 0.02 1.0"/>
+  </material>
+  <material name="arm_blue">
+    <color rgba="0.0 0.0 0.8 0.7"/>
   </material>
   <!-- ===================== -->
@@ -51,4 +57,5 @@
         <cylinder length="${l1}" radius="${r}"/>
       </geometry>
+      <material name="arm_blue"/>
     </visual>
     <collision>
@@ -79,4 +86,5 @@
         <cylinder length="${l2}" radius="${r}"/>
       </geometry>
+      <material name="arm_blue"/>
     </visual>
     <collision>
@@ -107,4 +115,5 @@
         <cylinder length="${l3}" radius="${r}"/>
       </geometry>
+      <material name="arm_blue"/>
     </visual>
     <collision>
@@ -135,4 +144,5 @@
         <cylinder length="${l4}" radius="0.025"/>
       </geometry>
+      <material name="arm_blue"/>
     </visual>
     <collision>
@@ -156,5 +166,5 @@
   <!-- LINK 5 -->
   <!-- ===================== -->
-  <!-- <link name="arm_link_5">
+  <link name="arm_link_5">
     <inertial>
       <origin xyz="0 0 ${l5_half}"/>
@@ -166,4 +176,5 @@
         <cylinder length="${l5}" radius="0.025"/>
       </geometry>
+      <material name="arm_blue"/>
     </visual>
     <collision>
@@ -173,13 +184,42 @@
       </geometry>
     </collision>
-  </link> -->
+  </link>
   <!-- Wrist roll joint (PERPENDICULAR) -->
-  <!-- <joint name="wrist_roll_joint" type="revolute">
+  <joint name="wrist_roll_joint" type="revolute">
     <parent link="arm_link_4"/>
     <child link="arm_link_5"/>
-    <origin xyz="0 0 ${l4}" rpy="1.5708 0 0"/>
-    <axis xyz="0 1 0"/>
+    <origin xyz="0 0 ${l4}" rpy="0 1.5708 0"/>
+    <axis xyz="1 0 0"/>
     <limit lower="-3.14" upper="3.14" effort="10" velocity="2.0"/>
-  </joint> -->
+  </joint>
+  <!-- ===================== -->
+  <!-- LINK 6 -->
+  <!-- ===================== -->
+  <link name="arm_link_6">
+    <inertial>
+      <origin xyz="0 0 ${l6_half}"/>
+      <xacro:cyl_inertia m="1.0" r="0.025" l="${l6}"/>
+    </inertial>
+    <visual>
+      <origin xyz="0 0 ${l6_half}"/>
+      <geometry>
+        <cylinder length="${l6}" radius="0.025"/>
+      </geometry>
+      <material name="arm_blue"/>
+    </visual>
+    <collision>
+      <origin xyz="0 0 ${l6_half}"/>
+      <geometry>
+        <cylinder length="${l6}" radius="0.025"/>
+      </geometry>
+    </collision>
+  </link>
+  <joint name="wrist_yaw_joint" type="revolute">
+    <parent link="arm_link_5"/>
+    <child link="arm_link_6"/>
+    <origin xyz="0 0 ${l5}" rpy="0 0 0"/>
+    <axis xyz="0 0 1"/>
+    <limit lower="-3.14" upper="3.14" effort="10" velocity="2.0"/>
+  </joint>
     <!-- ===================== -->
   <!-- END EFFECTOR -->
@@ -187,9 +227,13 @@
   <link name="tool0"/>
     <joint name="wrist_to_tool0" type="fixed">
-      <parent link="arm_link_4"/>
+      <parent link="arm_link_6"/>
       <child link="tool0"/>
       <!-- adjust xyz if needed -->
-      <origin xyz="0 0 ${l4}" rpy="0 0 0"/>
-    </joint>
+      <origin xyz="0 0 ${l6}" rpy="0 0 0"/>
+    </joint>
+    <!-- ===================== -->
+    <!-- SIMPLE GRIPPER -->
+    <!-- ===================== -->
+    <xacro:simple_gripper parent_link="tool0"/>
     <!-- ee_link : physical tool -->
   <link name="ee_link">
@@ -237,9 +281,21 @@
       <state_interface name="velocity"/>
     </joint>
-    <!-- <joint name="wrist_roll_joint">
-      <command_interface name="position"/>
-      <state_interface name="position"/>
-      <state_interface name="velocity"/>
-    </joint> -->
+    <joint name="wrist_roll_joint">
+      <command_interface name="position"/>
+      <state_interface name="position"/>
+      <state_interface name="velocity"/>
+    </joint>
+    <joint name="wrist_yaw_joint">
+      <command_interface name="position"/>
+      <state_interface name="position"/>
+      <state_interface name="velocity"/>
+    </joint>
+    <joint name="right_finger_joint">
+      <command_interface name="position"/>
+      <state_interface name="position"/>
+    </joint>
+    <joint name="left_finger_joint">
+      <state_interface name="position"/>
+    </joint>
     <joint name="FWRJ">
       <command_interface name="velocity"/>

File: ebot_description/models/ebot/ebot_description.xacro (robot description, xacro)
@@ -258,4 +258,9 @@
       </material>
     </visual>
+    <collision>
+      <geometry>
+        <cylinder length="0.04" radius="0.03"/>
+      </geometry>
+    </collision>
   </link>
   <joint name="lidar_joint" type="fixed">
@@ -273,4 +278,9 @@
       </material>
     </visual>
+    <collision>
+      <geometry>
+        <box size="0.10 0.015 0.008"/>
+      </geometry>
+    </collision>
   </link>
   <joint name="imu_joint" type="fixed">

Commit message: setup

File: arm_description/urdf/arm.xacro (robot description, xacro)
@@ -1,5 +1,5 @@
 <?xml version="1.0"?>
 <robot xmlns:xacro="http://www.ros.org/wiki/xacro">
-<xacro:include filename="$(find arm_description)/urdf/simple_gripper.xacro"/>
+<!-- <xacro:include filename="$(find arm_description)/urdf/simple_gripper.xacro"/> -->
   <xacro:macro name="ebot_arm">
   <!-- ===================== -->
@@ -235,5 +235,5 @@
     <!-- SIMPLE GRIPPER -->
     <!-- ===================== -->
-    <xacro:simple_gripper parent_link="tool0"/>
+    <!-- <xacro:simple_gripper parent_link="tool0"/> -->
     <!-- ee_link : physical tool -->
   <link name="ee_link">
@@ -257,6 +257,6 @@
   <ros2_control name="ArmSystem" type="system">
   <hardware>
-    <!-- <plugin>gz_ros2_control/GazeboSimSystem</plugin> -->
-    <plugin>mock_components/GenericSystem</plugin>
+    <plugin>gz_ros2_control/GazeboSimSystem</plugin>
+    <!-- <plugin>mock_components/GenericSystem</plugin> -->
     <param name="initial_positions">0 0 0 0</param>
   </hardware>

File: arm_description/urdf/simple_gripper.xacro (robot description, xacro)
@@ -34,5 +34,10 @@
         </geometry>
       </collision>
-    </link>
+      <inertia
+        ixx="1e-5" ixy="0.0" ixz="0.0"
+        iyy="1e-5" iyz="0.0"
+        izz="1e-5"/>
+    </inertial>
+      </link>
     <joint name="right_finger_joint" type="prismatic">
       <parent link="gripper_base_link"/>
@@ -56,4 +61,12 @@
         </geometry>
       </collision>
+      <inertial>
+        <origin xyz="0 0 0"/>
+        <mass value="0.05"/>
+        <inertia
+          ixx="1e-5" ixy="0.0" ixz="0.0"
+          iyy="1e-5" iyz="0.0"
+          izz="1e-5"/>
+      </inertial>
     </link>
     <joint name="left_finger_joint" type="prismatic">
