Commit message: added kdl cpp

File: arm_description/urdf/arm.xacro (robot description, xacro)
@@ -1,4 +1,5 @@
 <?xml version="1.0"?>
 <robot xmlns:xacro="http://www.ros.org/wiki/xacro">
+<!-- <xacro:include filename="$(find arm_description)/urdf/simple_gripper.xacro"/> -->
   <xacro:macro name="ebot_arm">
   <!-- ===================== -->
@@ -11,10 +12,12 @@
   <xacro:property name="l3" value="0.25"/>
   <xacro:property name="l4" value="0.05"/>
-  <xacro:property name="l5" value="0.10"/>
+  <!-- <xacro:property name="l5" value="0.05"/>
+  <xacro:property name="l6" value="0.05"/> -->
   <xacro:property name="l1_half" value="0.05"/>
   <xacro:property name="l2_half" value="0.15"/>
   <xacro:property name="l3_half" value="0.125"/>
   <xacro:property name="l4_half" value="0.025"/>
-  <xacro:property name="l5_half" value="0.05"/>
+  <!-- <xacro:property name="l5_half" value="0.025"/>
+  <xacro:property name="l6_half" value="0.025"/> -->
     <!-- ===================== -->
   <!-- MATERIALS -->
@@ -23,4 +26,7 @@
     <color rgba="0.02 0.02 0.02 1.0"/>
   </material>
+  <!-- <material name="arm_blue">
+    <color rgba="0.0 0.0 0.8 0.7"/>
+  </material> -->
   <!-- ===================== -->
   <!-- INERTIA MACRO -->
@@ -153,7 +159,4 @@
   <!-- LINK 5 -->
   <!-- ===================== -->
-  <!-- ===================== -->
-  <!-- LINK 5 -->
-  <!-- ===================== -->
   <!-- <link name="arm_link_5">
     <inertial>
@@ -178,9 +181,38 @@
     <parent link="arm_link_4"/>
     <child link="arm_link_5"/>
-    <origin xyz="0 0 ${l4}" rpy="1.5708 0 0"/>
-    <axis xyz="0 1 0"/>
+    <origin xyz="0 0 ${l4}" rpy="0 1.5708 0"/>
+    <axis xyz="1 0 0"/>
     <limit lower="-3.14" upper="3.14" effort="10" velocity="2.0"/>
   </joint> -->
-    <!-- ===================== -->
+ <!-- ===================== -->
+  <!-- LINK 6 -->
+  <!-- ===================== -->
+  <!-- <link name="arm_link_6">
+    <inertial>
+      <origin xyz="0 0 ${l6_half}"/>
+      <xacro:cyl_inertia m="1.0" r="0.025" l="${l6}"/>
+    </inertial>
+    <visual>
+      <origin xyz="0 0 ${l6_half}"/>
+      <geometry>
+        <cylinder length="${l6}" radius="0.025"/>
+      </geometry>
+      <material name="arm_blue"/>
+    </visual>
+    <collision>
+      <origin xyz="0 0 ${l6_half}"/>
+      <geometry>
+        <cylinder length="${l6}" radius="0.025"/>
+      </geometry>
+    </collision>
+  </link>
+  <joint name="wrist_yaw_joint" type="revolute">
+    <parent link="arm_link_5"/>
+    <child link="arm_link_6"/>
+    <origin xyz="0 0 ${l5}" rpy="0 0 0"/>
+    <axis xyz="0 0 1"/>
+    <limit lower="-3.14" upper="3.14" effort="10" velocity="2.0"/>
+  </joint> -->
+  <!-- ===================== -->
   <!-- END EFFECTOR -->
   <!-- ===================== -->
@@ -211,4 +243,8 @@
       <origin xyz="0.0 0 0"/>
     </joint>
+    <!-- ===================== -->
+    <!-- SIMPLE GRIPPER -->
+    <!-- ===================== -->
+    <!-- <xacro:simple_gripper parent_link="tool0"/> -->
   <ros2_control name="ArmSystem" type="system">
   <hardware>
@@ -242,4 +278,16 @@
       <state_interface name="velocity"/>
     </joint> -->
+    <!-- <joint name="wrist_yaw_joint">
+      <command_interface name="position"/>
+      <state_interface name="position"/>
+      <state_interface name="velocity"/>
+    </joint>
+    <joint name="right_finger_joint">
+      <command_interface name="position"/>
+      <state_interface name="position"/>
+    </joint>
+    <joint name="left_finger_joint">
+      <state_interface name="position"/>
+    </joint> -->
     <joint name="FWRJ">
       <command_interface name="velocity"/>

Commit message: arm haerdware pluging added

File: arm_description/urdf/arm.xacro (robot description, xacro)
@@ -249,27 +249,30 @@
   <ros2_control name="ArmSystem" type="system">
   <hardware>
+    <plugin>ebot_arm_hardware/ArmHardware</plugin>
+    <param name="port">/dev/ttyACM1</param>
+    <param name="baudrate">115200</param>
     <!-- <plugin>gz_ros2_control/GazeboSimSystem</plugin> -->
-    <plugin>mock_components/GenericSystem</plugin>
-    <param name="initial_positions">0 0 0 0</param>
+    <!-- <plugin>mock_components/GenericSystem</plugin> -->
+    <!-- <param name="initial_positions">0 0 0 0</param> -->
   </hardware>
     <joint name="base_rotation_joint">
       <command_interface name="position"/>
       <state_interface name="position"/>
-      <state_interface name="velocity"/>
+      <!-- <state_interface name="velocity"/> -->
     </joint>
     <joint name="shoulder_joint">
       <command_interface name="position"/>
       <state_interface name="position"/>
-      <state_interface name="velocity"/>
+      <!-- <state_interface name="velocity"/> -->
     </joint>
     <joint name="elbow_joint">
       <command_interface name="position"/>
       <state_interface name="position"/>
-      <state_interface name="velocity"/>
+      <!-- <state_interface name="velocity"/> -->
     </joint>
     <joint name="wrist_joint">
       <command_interface name="position"/>
       <state_interface name="position"/>
-      <state_interface name="velocity"/>
+      <!-- <state_interface name="velocity"/> -->
     </joint>
     <!-- <joint name="wrist_roll_joint">
@@ -290,5 +293,5 @@
       <state_interface name="position"/>
     </joint> -->
-    <joint name="FWRJ">
+    <!-- <joint name="FWRJ">
       <command_interface name="velocity"/>
       <state_interface name="position"/>
@@ -299,5 +302,5 @@
       <state_interface name="position"/>
       <state_interface name="velocity"/>
-    </joint>
+    </joint> -->
   </ros2_control>
   </xacro:macro>

File: ebot_description/models/ebot/ebot_description.xacro (robot description, xacro)
@@ -98,5 +98,7 @@
     <parent link="ebot_base"/>
     <child link="FWR"/>
-    <axis xyz="1 0 0"/>
+    <axis xyz="0 1 0"/>
+    <limit effort="10.0" velocity="20.0"/>
+    <dynamics damping="0.1" friction="0.0"/>
   </joint>
   <!-- Front Left -->
@@ -125,9 +127,12 @@
     <parent link="ebot_base"/>
     <child link="FWL"/>
-    <axis xyz="1 0 0"/>
+    <axis xyz="0 1 0"/>
+    <limit effort="10.0" velocity="20.0"/>
+    <dynamics damping="0.1" friction="0.0"/>
   </joint>
   <!-- ===================== -->
   <!-- TRANSMISSIONS -->
   <!-- ===================== -->
+<!--
   <transmission name="FWR_trans">
     <type>transmission_interface/SimpleTransmission</type>
@@ -147,5 +152,5 @@
       <mechanicalReduction>1</mechanicalReduction>
     </actuator>
-  </transmission>
+  </transmission> -->
   <!-- ===================== -->
   <!-- OMNI CASTERS (SWIVEL + ROLL) -->

Commit message: arm hardware

File: arm_description/urdf/arm.xacro (robot description, xacro)
@@ -8,4 +8,7 @@
   <xacro:property name="r" value="0.03"/>
   <xacro:property name="m" value="2.0"/>
+  <xacro:property name="m1" value="1.8"/>   <!-- base link -->
+  <xacro:property name="m2" value="1.5"/>   <!-- shoulder link -->
+  <xacro:property name="m3" value="1.0"/>   <!-- elbow link -->
   <xacro:property name="l1" value="0.10"/>
   <xacro:property name="l2" value="0.30"/>
@@ -35,7 +38,7 @@
     <mass value="${m}"/>
     <inertia
-      ixx="${m*(3*r*r + l*l)/12}"
-      iyy="${m*(3*r*r + l*l)/12}"
-      izz="${m*(r*r)/2}"
+      ixx="${0.7 * m*(3*r*r + l*l)/12}"
+      iyy="${0.7 * m*(3*r*r + l*l)/12}"
+      izz="${0.7 * m*(r*r)/2}"
       ixy="0" ixz="0" iyz="0"/>
   </xacro:macro>
@@ -50,5 +53,5 @@
     <inertial>
       <origin xyz="0 0 ${l1_half}"/>
-      <xacro:cyl_inertia m="${m}" r="${r}" l="${l1}"/>
+      <xacro:cyl_inertia m="${m1}" r="${r}" l="${l1}"/>
     </inertial>
     <visual>
@@ -77,6 +80,6 @@
   <link name="arm_link_2">
     <inertial>
-      <origin xyz="0 0 ${l2_half}"/>
-      <xacro:cyl_inertia m="${m}" r="${r}" l="${l2}"/>
+      <origin xyz="0 0 ${0.12}"/>
+      <xacro:cyl_inertia m="${m2}" r="${r}" l="${l2}"/>
     </inertial>
     <visual>
@@ -98,5 +101,5 @@
     <origin xyz="0 0 ${l1}"/>
     <axis xyz="0 1 0"/>
-    <limit lower="-1.57" upper="1.57" effort="20" velocity="1.5"/>
+    <limit lower="-1.57" upper="1.57" effort="36" velocity="1.5"/>
   </joint>
   <!-- ===================== -->
@@ -105,6 +108,6 @@
   <link name="arm_link_3">
     <inertial>
-      <origin xyz="0 0 ${l3_half}"/>
-      <xacro:cyl_inertia m="${m}" r="${r}" l="${l3}"/>
+      <origin xyz="0 0 ${0.09}"/>
+      <xacro:cyl_inertia m="${m3}" r="${r}" l="${l3}"/>
     </inertial>
     <visual>
@@ -249,8 +252,8 @@
   <ros2_control name="ArmSystem" type="system">
   <hardware>
-    <plugin>ebot_arm_hardware/ArmHardware</plugin>
+    <!-- <plugin>ebot_arm_hardware/ArmHardware</plugin>
     <param name="port">/dev/ttyACM1</param>
-    <param name="baudrate">115200</param>
-    <!-- <plugin>gz_ros2_control/GazeboSimSystem</plugin> -->
+    <param name="baudrate">115200</param> -->
+    <plugin>gz_ros2_control/GazeboSimSystem</plugin>
     <!-- <plugin>mock_components/GenericSystem</plugin> -->
     <!-- <param name="initial_positions">0 0 0 0</param> -->
@@ -259,20 +262,20 @@
       <command_interface name="position"/>
       <state_interface name="position"/>
-      <!-- <state_interface name="velocity"/> -->
+      <state_interface name="velocity"/>
     </joint>
     <joint name="shoulder_joint">
       <command_interface name="position"/>
       <state_interface name="position"/>
-      <!-- <state_interface name="velocity"/> -->
+      <state_interface name="velocity"/>
     </joint>
     <joint name="elbow_joint">
       <command_interface name="position"/>
       <state_interface name="position"/>
-      <!-- <state_interface name="velocity"/> -->
+      <state_interface name="velocity"/>
     </joint>
     <joint name="wrist_joint">
       <command_interface name="position"/>
       <state_interface name="position"/>
-      <!-- <state_interface name="velocity"/> -->
+      <state_interface name="velocity"/>
     </joint>
     <!-- <joint name="wrist_roll_joint">
@@ -293,5 +296,5 @@
       <state_interface name="position"/>
     </joint> -->
-    <!-- <joint name="FWRJ">
+    <joint name="FWRJ">
       <command_interface name="velocity"/>
       <state_interface name="position"/>
@@ -302,5 +305,5 @@
       <state_interface name="position"/>
       <state_interface name="velocity"/>
-    </joint> -->
+    </joint>
   </ros2_control>
   </xacro:macro>

Commit message: 6d0f

File: arm_description/urdf/arm.xacro (robot description, xacro)
@@ -1,5 +1,5 @@
 <?xml version="1.0"?>
 <robot xmlns:xacro="http://www.ros.org/wiki/xacro">
-<!-- <xacro:include filename="$(find arm_description)/urdf/simple_gripper.xacro"/> -->
+<xacro:include filename="$(find arm_description)/urdf/simple_gripper.xacro"/>
   <xacro:macro name="ebot_arm">
   <!-- ===================== -->
@@ -15,12 +15,12 @@
   <xacro:property name="l3" value="0.25"/>
   <xacro:property name="l4" value="0.05"/>
-  <!-- <xacro:property name="l5" value="0.05"/>
-  <xacro:property name="l6" value="0.05"/> -->
+  <xacro:property name="l5" value="0.05"/>
+  <xacro:property name="l6" value="0.05"/>
   <xacro:property name="l1_half" value="0.05"/>
   <xacro:property name="l2_half" value="0.15"/>
   <xacro:property name="l3_half" value="0.125"/>
   <xacro:property name="l4_half" value="0.025"/>
-  <!-- <xacro:property name="l5_half" value="0.025"/>
-  <xacro:property name="l6_half" value="0.025"/> -->
+  <xacro:property name="l5_half" value="0.025"/>
+  <xacro:property name="l6_half" value="0.025"/>
     <!-- ===================== -->
   <!-- MATERIALS -->
@@ -29,7 +29,7 @@
     <color rgba="0.02 0.02 0.02 1.0"/>
   </material>
-  <!-- <material name="arm_blue">
+  <material name="arm_blue">
     <color rgba="0.0 0.0 0.8 0.7"/>
-  </material> -->
+  </material>
   <!-- ===================== -->
   <!-- INERTIA MACRO -->
@@ -99,5 +99,5 @@
     <parent link="arm_link_1"/>
     <child link="arm_link_2"/>
-    <origin xyz="0 0 ${l1}"/>
+    <origin xyz="0 0.06 ${l1}"/>
     <axis xyz="0 1 0"/>
     <limit lower="-1.57" upper="1.57" effort="36" velocity="1.5"/>
@@ -127,5 +127,5 @@
     <parent link="arm_link_2"/>
     <child link="arm_link_3"/>
-    <origin xyz="0 0 ${l2}"/>
+    <origin xyz="0 -0.06 ${l2}"/>
     <axis xyz="0 1 0"/>
     <limit lower="0.00" upper="3.1" effort="15" velocity="1.5"/>
@@ -155,5 +155,5 @@
     <parent link="arm_link_3"/>
     <child link="arm_link_4"/>
-    <origin xyz="0 0 ${l3}"/>
+    <origin xyz="0 0.05 ${l3}"/>
     <axis xyz="0 1 0"/>
     <limit lower="-3.14" upper="3.14" effort="10" velocity="2.0"/>
@@ -162,5 +162,5 @@
   <!-- LINK 5 -->
   <!-- ===================== -->
-  <!-- <link name="arm_link_5">
+  <link name="arm_link_5">
     <inertial>
       <origin xyz="0 0 ${l5_half}"/>
@@ -179,7 +179,7 @@
       </geometry>
     </collision>
-  </link> -->
+  </link>
   <!-- Wrist roll joint (PERPENDICULAR) -->
-  <!-- <joint name="wrist_roll_joint" type="revolute">
+  <joint name="wrist_roll_joint" type="revolute">
     <parent link="arm_link_4"/>
     <child link="arm_link_5"/>
@@ -187,9 +187,9 @@
     <axis xyz="1 0 0"/>
     <limit lower="-3.14" upper="3.14" effort="10" velocity="2.0"/>
-  </joint> -->
+  </joint>
  <!-- ===================== -->
   <!-- LINK 6 -->
   <!-- ===================== -->
-  <!-- <link name="arm_link_6">
+  <link name="arm_link_6">
     <inertial>
       <origin xyz="0 0 ${l6_half}"/>
@@ -216,5 +216,5 @@
     <axis xyz="0 0 1"/>
     <limit lower="-3.14" upper="3.14" effort="10" velocity="2.0"/>
-  </joint> -->
+  </joint>
   <!-- ===================== -->
   <!-- END EFFECTOR -->
@@ -222,8 +222,8 @@
   <link name="tool0"/>
     <joint name="wrist_to_tool0" type="fixed">
-      <parent link="arm_link_4"/>
+      <parent link="arm_link_6"/>
       <child link="tool0"/>
       <!-- adjust xyz if needed -->
-      <origin xyz="0 0 ${l4}" rpy="0 0 0"/>
+      <origin xyz="0 0 ${l6}" rpy="0 0 0"/>
     </joint>
     <!-- ee_link : physical tool -->
@@ -249,5 +249,5 @@
     <!-- SIMPLE GRIPPER -->
     <!-- ===================== -->
-    <!-- <xacro:simple_gripper parent_link="tool0"/> -->
+    <xacro:simple_gripper parent_link="tool0"/>
   <ros2_control name="ArmSystem" type="system">
   <hardware>
@@ -255,6 +255,6 @@
     <param name="port">/dev/ttyACM1</param>
     <param name="baudrate">115200</param> -->
-    <plugin>gz_ros2_control/GazeboSimSystem</plugin>
-    <!-- <plugin>mock_components/GenericSystem</plugin> -->
+    <!-- <plugin>gz_ros2_control/GazeboSimSystem</plugin> -->
+    <plugin>mock_components/GenericSystem</plugin>
     <!-- <param name="initial_positions">0 0 0 0</param> -->
   </hardware>
@@ -279,10 +279,10 @@
       <state_interface name="velocity"/>
     </joint>
-    <!-- <joint name="wrist_roll_joint">
-      <command_interface name="position"/>
-      <state_interface name="position"/>
-      <state_interface name="velocity"/>
-    </joint> -->
-    <!-- <joint name="wrist_yaw_joint">
+    <joint name="wrist_roll_joint">
+      <command_interface name="position"/>
+      <state_interface name="position"/>
+      <state_interface name="velocity"/>
+    </joint>
+    <joint name="wrist_yaw_joint">
       <command_interface name="position"/>
       <state_interface name="position"/>
@@ -295,5 +295,5 @@
     <joint name="left_finger_joint">
       <state_interface name="position"/>
-    </joint> -->
+    </joint>
     <joint name="FWRJ">
       <command_interface name="velocity"/>

File: arm_description/urdf/simple_gripper.xacro (robot description, xacro)
@@ -6,7 +6,7 @@
   <xacro:macro name="simple_gripper" params="parent_link">
     <!-- Bigger parameters -->
-    <xacro:property name="finger_length" value="0.105"/>
+    <xacro:property name="finger_length" value="0.035"/>
     <xacro:property name="finger_width"  value="0.015"/>
-    <xacro:property name="finger_height" value="0.03"/>
+    <xacro:property name="finger_height" value="0.105"/>
     <xacro:property name="finger_offset" value="0.06"/>
     <xacro:property name="finger_travel" value="0.05"/>
@@ -38,10 +38,9 @@
         iyy="1e-5" iyz="0.0"
         izz="1e-5"/>
-    </inertial>
-      </link>
+    </link>
     <joint name="right_finger_joint" type="prismatic">
       <parent link="gripper_base_link"/>
       <child link="right_finger"/>
-      <origin xyz="0 -${finger_offset} 0"/>
+      <origin xyz="0 -${finger_offset} 0.05"/>
       <axis xyz="0 1 0"/>
       <limit lower="0.0" upper="${finger_travel}" effort="20" velocity="0.1"/>
@@ -73,5 +72,5 @@
       <parent link="gripper_base_link"/>
       <child link="left_finger"/>
-      <origin xyz="0 ${finger_offset} 0"/>
+      <origin xyz="0 ${finger_offset} 0.05"/>
       <axis xyz="0 -1 0"/>
       <limit lower="0.0" upper="${finger_travel}" effort="20" velocity="0.1"/>

Commit message: moveo arm on ebot

File: arm_description/urdf/arm.xacro (robot description, xacro)
@@ -255,6 +255,6 @@
     <param name="port">/dev/ttyACM1</param>
     <param name="baudrate">115200</param> -->
-    <!-- <plugin>gz_ros2_control/GazeboSimSystem</plugin> -->
-    <plugin>mock_components/GenericSystem</plugin>
+    <plugin>gz_ros2_control/GazeboSimSystem</plugin>
+    <!-- <plugin>mock_components/GenericSystem</plugin> -->
     <!-- <param name="initial_positions">0 0 0 0</param> -->
   </hardware>

File: arm_description/urdf/simple_gripper.xacro (robot description, xacro)
@@ -34,8 +34,12 @@
         </geometry>
       </collision>
-      <inertia
-        ixx="1e-5" ixy="0.0" ixz="0.0"
-        iyy="1e-5" iyz="0.0"
-        izz="1e-5"/>
+      <inertial>
+        <origin xyz="0 0 0"/>
+        <mass value="0.05"/>
+        <inertia
+          ixx="1e-5" ixy="0" ixz="0"
+          iyy="1e-5" iyz="0"
+          izz="1e-5"/>
+      </inertial>
     </link>
     <joint name="right_finger_joint" type="prismatic">

File: ebot_description/models/ebot/ebot_description.xacro (robot description, xacro)
@@ -3,7 +3,8 @@
   <xacro:arg name="use_gazebo" default="true"/>
   <xacro:include filename="$(find ebot_description)/models/ebot/ebot.gazebo" />
-  <xacro:include filename="$(find arm_description)/urdf/arm.xacro" />
+  <!-- <xacro:include filename="$(find arm_description)/urdf/arm.xacro" /> -->
   <xacro:include filename="$(find ebot_description)/models/ebot/ebot_gazebo_control.xacro"/>
-  <xacro:ebot_arm/>
+  <xacro:include filename="$(find moveo_description)/urdf/moveo_urdf.urdf.xacro"/>
+  <xacro:moveo_arm prefix="moveo_"/>
   <!-- ===================== -->
   <!-- PROPERTIES -->
@@ -67,6 +68,6 @@
   <joint name="arm_mount_joint" type="fixed">
     <parent link="ebot_base"/>
-    <child link="arm_base_link"/>
-    <origin xyz="0 0 0.12" rpy="0 0 0"/>
+    <child link="moveo_base_link"/>
+    <origin xyz="0 0 0.0" rpy="0 0 -1.5708"/>
   </joint>
   <!-- ===================== -->
