Commit message: hardware plugin added

File: ebot_description/models/ebot/ebot_ros2_control.xacro (robot description, xacro)
@@ -4,9 +4,9 @@
     <ros2_control name="EbotSystem" type="system">
     <hardware>
-        <!-- <plugin>ebot_arm_hardware/ArmHardware</plugin>
-        <param name="port">/dev/ttyACM1</param>
-        <param name="baudrate">115200</param> -->
+        <plugin>moveo_hardware/MoveoSystem</plugin>
+        <param name="port">/dev/ttyACM0</param>
+        <param name="baudrate">115200</param>
         <!-- <plugin>gz_ros2_control/GazeboSimSystem</plugin> -->
-        <plugin>mock_components/GenericSystem</plugin>
+        <!-- <plugin>mock_components/GenericSystem</plugin> -->
         <!-- <param name="initial_positions">0 0 0 0</param> -->
     </hardware>
@@ -14,27 +14,27 @@
         <command_interface name="position"/>
         <state_interface name="position"/>
-        <state_interface name="velocity"/>
+        <!-- <state_interface name="velocity"/> -->
         </joint>
         <joint name="Joint_2">
         <command_interface name="position"/>
         <state_interface name="position"/>
-        <state_interface name="velocity"/>
+        <!-- <state_interface name="velocity"/> -->
         </joint>
         <joint name="Joint_3">
         <command_interface name="position"/>
         <state_interface name="position"/>
-        <state_interface name="velocity"/>
+        <!-- <state_interface name="velocity"/> -->
         </joint>
         <joint name="Joint_4">
         <command_interface name="position"/>
         <state_interface name="position"/>
-        <state_interface name="velocity"/>
+        <!-- <state_interface name="velocity"/> -->
         </joint>
         <joint name="Joint_5">
         <command_interface name="position"/>
         <state_interface name="position"/>
-        <state_interface name="velocity"/>
+        <!-- <state_interface name="velocity"/>/ -->
         </joint>
-        <joint name="Gripper_Servo_Gear_Joint">
+        <!-- <joint name="Gripper_Servo_Gear_Joint">
         <command_interface name="position"/>
         <state_interface name="position"/>
@@ -53,5 +53,5 @@
         <state_interface name="position"/>
         <state_interface name="velocity"/>
-        </joint>
+        </joint> -->
     </ros2_control>
   </xacro:macro>
