Commit message: movit applied

File: ebot_description/models/ebot/ebot_description.xacro (robot description, xacro)
@@ -2,4 +2,5 @@
 <robot name="ebot" xmlns:xacro="http://www.ros.org/wiki/xacro">
   <xacro:include filename="$(find ebot_description)/models/ebot/ebot.gazebo" />
+  <xacro:include filename="$(find open_manipulator_description)/urdf/open_manipulator_x/open_manipulator_x_arm.urdf.xacro"/>
   <!-- ===================== -->
   <!-- PROPERTIES -->
@@ -48,7 +49,7 @@
     </visual>
     <collision>
-      <origin xyz="0 0 0.12"/>
-      <geometry>
-        <box size="0.585 0.50 0.25"/>
+      <origin xyz="0 0 0.07"/>
+      <geometry>
+        <box size="0.510 0.30 0.10"/>
       </geometry>
     </collision>
@@ -57,4 +58,10 @@
     <parent link="ebot_base_link"/>
     <child link="ebot_base"/>
+  </joint>
+  <xacro:open_manipulator_x prefix="arm_"/>
+  <joint name="ebot_to_arm_joint" type="fixed">
+    <parent link="ebot_base"/>
+    <child link="arm_link1"/>
+    <origin xyz="0 0 0.30" rpy="0 0 0"/>
   </joint>
   <!-- ===================== -->

Commit message: ros2 controller to arm

File: ebot_description/models/ebot/ebot_description.xacro (robot description, xacro)
@@ -2,4 +2,5 @@
 <robot name="ebot" xmlns:xacro="http://www.ros.org/wiki/xacro">
   <xacro:include filename="$(find ebot_description)/models/ebot/ebot.gazebo" />
+  <xacro:include filename="$(find arm_description)/urdf/arm.xacro" />
   <!-- ===================== -->
   <!-- PROPERTIES -->
@@ -59,4 +60,12 @@
   </joint>
   <!-- ===================== -->
+  <!-- ARM MOUNT -->
+  <!-- ===================== -->
+  <joint name="arm_mount_joint" type="fixed">
+    <parent link="ebot_base"/>
+    <child link="arm_base_link"/>
+    <origin xyz="0 0 0.25" rpy="0 0 0"/>
+  </joint>
+  <!-- ===================== -->
   <!-- DRIVE WHEELS -->
   <!-- ===================== -->

Commit message: cartesian servo with KDL arm

File: ebot_description/models/ebot/ebot_description.xacro (robot description, xacro)
@@ -98,5 +98,5 @@
     <parent link="ebot_base"/>
     <child link="FWR"/>
-    <axis xyz="0 1 0"/>
+    <axis xyz="1 0 0"/>
   </joint>
   <!-- Front Left -->
@@ -125,5 +125,5 @@
     <parent link="ebot_base"/>
     <child link="FWL"/>
-    <axis xyz="0 1 0"/>
+    <axis xyz="1 0 0"/>
   </joint>
   <!-- ===================== -->

Commit message: mapping done

File: ebot_description/models/ebot/ebot_description.xacro (robot description, xacro)
@@ -227,5 +227,5 @@
   </link>
   <joint name="lidar_joint" type="fixed">
-    <origin xyz="0.2055 0 0.15"/>
+    <origin xyz="0.12 0.075 0.15"/>
     <parent link="ebot_base"/>
     <child link="laser"/>

Commit message: implementing imu+magnetometer

File: ebot_description/models/ebot/ebot_description.xacro (robot description, xacro)
@@ -227,5 +227,5 @@
   </link>
   <joint name="lidar_joint" type="fixed">
-    <origin xyz="0.12 0.075 0.15"/>
+    <origin xyz="0.12 0.075 0.31"/>
     <parent link="ebot_base"/>
     <child link="laser"/>

Commit message: starting on mobile nav2 planner

File: ebot_description/models/ebot/ebot_description.xacro (robot description, xacro)
@@ -227,5 +227,5 @@
   </link>
   <joint name="lidar_joint" type="fixed">
-    <origin xyz="0.12 0.075 0.31"/>
+    <origin xyz="0.14 0.055 0.31"/>
     <parent link="ebot_base"/>
     <child link="laser"/>

Commit message: changed urdf

File: ebot_description/models/ebot/ebot_description.xacro (robot description, xacro)
@@ -216,4 +216,5 @@
   <!-- SENSORS -->
   <!-- ===================== -->
+  <!--laser-->
   <link name="laser">
     <visual>
@@ -231,4 +232,37 @@
     <child link="laser"/>
   </joint>
+  <!--3d lidar-->
+  <link name="3d_laser">
+    <visual>
+      <geometry>
+        <cylinder length="0.02" radius="0.01"/>
+      </geometry>
+            <material name="wheel_black">
+        <color rgba="0.02 0.02 0.02 1.0"/>
+      </material>
+    </visual>
+  </link>
+  <joint name="3d_lidar_joint" type="fixed">
+    <origin xyz="0.12 0.075 0.31"/>
+    <parent link="ebot_base"/>
+    <child link="3d_laser"/>
+  </joint>
+  <!--imu on lidar-->
+  <link name="lidar_imu_link">
+    <visual>
+      <geometry>
+        <box size="0.10 0.015 0.008"/>
+      </geometry>
+            <material name="wheel_black">
+        <color rgba="0.02 0.02 0.02 1.0"/>
+      </material>
+    </visual>
+  </link>
+  <joint name="lidar_imu_joint" type="fixed">
+    <origin xyz="0.12 0.075 0.31"/>
+    <parent link="ebot_base"/>
+    <child link="lidar_imu_link"/>
+  </joint>
+  <!--bot imu-->
   <link name="imu_link">
     <visual>

Commit message: imu error resolved

File: ebot_description/models/ebot/ebot_description.xacro (robot description, xacro)
@@ -244,10 +244,10 @@
   </link>
   <joint name="3d_lidar_joint" type="fixed">
-    <origin xyz="0.12 0.075 0.31"/>
+    <origin xyz="0.14 0.055 0.31"/>
     <parent link="ebot_base"/>
     <child link="3d_laser"/>
   </joint>
   <!--imu on lidar-->
-  <link name="lidar_imu_link">
+  <!-- <link name="lidar_imu_link">
     <visual>
       <geometry>
@@ -263,5 +263,5 @@
     <parent link="ebot_base"/>
     <child link="lidar_imu_link"/>
-  </joint>
+  </joint> -->
   <!--bot imu-->
   <link name="imu_link">
@@ -280,3 +280,19 @@
     <child link="imu_link"/>
   </joint>
+  <link name="camera">
+    <visual>
+     <origin rpy="0 1.5708 0"/>
+      <geometry>
+        <cylinder length="0.04" radius="0.01"/>
+      </geometry>
+            <material name="wheel_black">
+        <color rgba="0.02 0.02 0.02 1.0"/>
+      </material>
+    </visual>
+  </link>
+  <joint name="camera_joint" type="fixed">
+    <origin xyz="0.14 0.052 0.24"/>
+    <parent link="ebot_base"/>
+    <child link="camera"/>
+  </joint>
 </robot>

Commit message: moveo arm setup

File: ebot_description/models/ebot/ebot_description.xacro (robot description, xacro)
@@ -6,4 +6,5 @@
   <xacro:include filename="$(find ebot_description)/models/ebot/ebot_gazebo_control.xacro"/>
   <xacro:include filename="$(find moveo_description)/urdf/moveo_urdf.urdf.xacro"/>
+  <xacro:include filename="$(find ebot_description)/models/ebot/ebot_ros2_control.xacro"/>
   <xacro:moveo_arm prefix="moveo_"/>
   <!-- ===================== -->
@@ -285,4 +286,5 @@
     <child link="imu_link"/>
   </joint>
+<xacro:ebot_ros2_control/>
 <xacro:ebot_gazebo_ros2_control/>
 </robot>

File: moveo_description/urdf/moveo_urdf.urdf.xacro (robot description, xacro)
@@ -344,104 +344,4 @@
         <mimic joint="Gripper_Idol_Gear_Joint" multiplier="1" offset="0" />
     </joint>
-  <gazebo>
-    <plugin filename="libgazebo_ros_control.so" name="gazebo_ros_control">
-      <robotNamespace>/moveo_description</robotNamespace>
-      <robotSimType>gazebo_ros_control/DefaultRobotHWSim</robotSimType>
-      <legacyModeNS>true</legacyModeNS>
-    </plugin>
-  </gazebo>
-    <transmission name="trans1">
-      <type>transmission_interface/SimpleTransmission</type>
-      <joint name="Joint_1">
-        <hardwareInterface>hardware_interface/EffortJointInterface</hardwareInterface>
-      </joint>
-      <actuator name="motor1">
-        <mechanicalReduction>1</mechanicalReduction>
-      </actuator>
-    </transmission>
-    <transmission name="trans2">
-      <type>transmission_interface/SimpleTransmission</type>
-      <joint name="Joint_2">
-        <hardwareInterface>hardware_interface/EffortJointInterface</hardwareInterface>
-      </joint>
-      <actuator name="motor2">
-        <mechanicalReduction>1</mechanicalReduction>
-      </actuator>
-    </transmission>
-    <transmission name="trans3">
-      <type>transmission_interface/SimpleTransmission</type>
-      <joint name="Joint_3">
-        <hardwareInterface>hardware_interface/EffortJointInterface</hardwareInterface>
-      </joint>
-      <actuator name="motor3">
-        <mechanicalReduction>1</mechanicalReduction>
-      </actuator>
-    </transmission>
-    <transmission name="trans4">
-      <type>transmission_interface/SimpleTransmission</type>
-      <joint name="Joint_4">
-        <hardwareInterface>hardware_interface/EffortJointInterface</hardwareInterface>
-      </joint>
-      <actuator name="motor4">
-        <mechanicalReduction>1</mechanicalReduction>
-      </actuator>
-    </transmission>
-    <transmission name="trans5">
-      <type>transmission_interface/SimpleTransmission</type>
-      <joint name="Joint_5">
-        <hardwareInterface>hardware_interface/EffortJointInterface</hardwareInterface>
-      </joint>
-      <actuator name="motor5">
-        <mechanicalReduction>1</mechanicalReduction>
-      </actuator>
-    </transmission>
-    <transmission name="trans6">
-      <type>transmission_interface/SimpleTransmission</type>
-      <joint name="Gripper_Servo_Gear_Joint">
-        <hardwareInterface>hardware_interface/EffortJointInterface</hardwareInterface>
-      </joint>
-      <actuator name="motor6">
-        <mechanicalReduction>1</mechanicalReduction>
-      </actuator>
-    </transmission>
-    <transmission name="trans7">
-      <type>transmission_interface/SimpleTransmission</type>
-      <joint name="Gripper_Idol_Gear_Joint">
-        <hardwareInterface>hardware_interface/EffortJointInterface</hardwareInterface>
-      </joint>
-      <actuator name="motor7">
-        <mechanicalReduction>1</mechanicalReduction>
-      </actuator>
-    </transmission>
-  <gazebo>
-    <plugin filename="libroboticsgroup_gazebo_mimic_joint_plugin.so" name="mimic_moveo_1">
-        <joint>Gripper_Servo_Gear_Joint</joint>
-        <mimicJoint>Tip_Gripper_Servo_Joint</mimicJoint>
-        <multiplier>1.0</multiplier>
-        <offset>0.0</offset>
-	<hasPID/>
-    </plugin>
-    <plugin filename="libroboticsgroup_gazebo_mimic_joint_plugin.so" name="mimic_moveo_2">
-        <joint>Gripper_Idol_Gear_Joint</joint>
-        <mimicJoint>Tip_Gripper_Idol_Joint</mimicJoint>
-        <multiplier>-1.0</multiplier>
-        <offset>0.0</offset>
-<hasPID/>
-    </plugin>
-    <plugin filename="libroboticsgroup_gazebo_mimic_joint_plugin.so" name="mimic_moveo_3">
-        <joint>Gripper_Servo_Gear_Joint</joint>
-        <mimicJoint>Pivot_Arm_Gripper_Servo_Joint</mimicJoint>
-        <multiplier>1.0</multiplier>
-        <offset>0.0</offset>
-<hasPID/>
-    </plugin>
-    <plugin filename="libroboticsgroup_gazebo_mimic_joint_plugin.so" name="mimic_moveo_4">
-        <joint>Gripper_Idol_Gear_Joint</joint>
-        <mimicJoint>Pivot_Arm_Gripper_Idol_Joint</mimicJoint>
-        <multiplier>1.0</multiplier>
-        <offset>0.0</offset>
-<hasPID/>
-</plugin>
-</gazebo>
 </xacro:macro>
 </robot>

Commit message: gazebo sim check and lidar added

File: ebot_description/models/ebot/ebot_description.xacro (robot description, xacro)
@@ -42,5 +42,5 @@
     <inertial>
       <origin xyz="0 0 0.12"/>
-      <xacro:box_inertia b_mass="${base_mass}" b_x="0.585" b_y="0.50" b_z="0.25"/>
+      <xacro:box_inertia b_mass="${base_mass}" b_x="0.510" b_y="0.30" b_z="0.10"/>
     </inertial>
     <visual>
@@ -56,5 +56,5 @@
       <origin xyz="0 0 0.12"/>
       <geometry>
-        <box size="0.585 0.50 0.25"/>
+        <box size="0.510 0.30 0.10"/>
       </geometry>
     </collision>
@@ -78,10 +78,10 @@
   <link name="FWR">
     <inertial>
-      <xacro:cylinder_inertia c_mass="${wheel_mass}" r="0.08" l="0.05"/>
+      <xacro:cylinder_inertia c_mass="${wheel_mass}" r="0.0625" l="0.05"/>
     </inertial>
     <visual>
       <origin rpy="1.5708 0 0"/>
       <geometry>
-        <cylinder length="0.05" radius="0.08"/>
+        <cylinder length="0.05" radius="0.0625"/>
       </geometry>
       <material name="wheel_black">
@@ -92,10 +92,10 @@
       <origin rpy="1.5708 0 0"/>
       <geometry>
-        <cylinder length="0.05" radius="0.08"/>
+        <cylinder length="0.05" radius="0.0625"/>
       </geometry>
     </collision>
   </link>
   <joint name="FWRJ" type="continuous">
-    <origin xyz="0 -0.20 0.045"/>
+    <origin xyz="0 -0.19 0.045"/>
     <parent link="ebot_base"/>
     <child link="FWR"/>
@@ -107,10 +107,10 @@
   <link name="FWL">
     <inertial>
-      <xacro:cylinder_inertia c_mass="${wheel_mass}" r="0.08" l="0.05"/>
+      <xacro:cylinder_inertia c_mass="${wheel_mass}" r="0.0625" l="0.05"/>
     </inertial>
     <visual>
       <origin rpy="1.5708 0 0"/>
       <geometry>
-        <cylinder length="0.05" radius="0.08"/>
+        <cylinder length="0.05" radius="0.0625"/>
       </geometry>
      <material name="wheel_black">
@@ -121,10 +121,10 @@
       <origin rpy="1.5708 0 0"/>
       <geometry>
-        <cylinder length="0.05" radius="0.08"/>
+        <cylinder length="0.05" radius="0.0625"/>
       </geometry>
     </collision>
   </link>
   <joint name="FWLJ" type="continuous">
-    <origin xyz="0 0.20 0.045"/>
+    <origin xyz="0 0.19 0.045"/>
     <parent link="ebot_base"/>
     <child link="FWL"/>
@@ -165,16 +165,16 @@
   <visual>
     <geometry>
-      <sphere radius="0.015"/>
-    </geometry>
-    <material name="wheel_black"/>
-  </visual>
-  <collision>
-    <geometry>
-      <sphere radius="0.015"/>
+      <sphere radius="0.010"/>
+    </geometry>
+    <material name="wheel_black"/>
+  </visual>
+  <collision>
+    <geometry>
+      <sphere radius="0.010"/>
     </geometry>
   </collision>
 </link>
 <joint name="BC_FRONT_J" type="fixed">
-  <origin xyz="0.20 0.1 -0.0200"/>
+  <origin xyz="0.20 0.1 -0.0030"/>
   <parent link="ebot_base"/>
   <child link="BC_FRONT"/>
@@ -184,16 +184,16 @@
   <visual>
     <geometry>
-      <sphere radius="0.015"/>
-    </geometry>
-    <material name="wheel_black"/>
-  </visual>
-  <collision>
-    <geometry>
-      <sphere radius="0.015"/>
+      <sphere radius="0.010"/>
+    </geometry>
+    <material name="wheel_black"/>
+  </visual>
+  <collision>
+    <geometry>
+      <sphere radius="0.010"/>
     </geometry>
   </collision>
 </link>
 <joint name="BC_BACK_J" type="fixed">
-  <origin xyz="-0.19 0.1 -0.0200"/>
+  <origin xyz="-0.19 0.1 -0.0030"/>
   <parent link="ebot_base"/>
   <child link="BC_BACK"/>
@@ -203,16 +203,16 @@
   <visual>
     <geometry>
-      <sphere radius="0.015"/>
-    </geometry>
-    <material name="wheel_black"/>
-  </visual>
-  <collision>
-    <geometry>
-      <sphere radius="0.015"/>
+      <sphere radius="0.010"/>
+    </geometry>
+    <material name="wheel_black"/>
+  </visual>
+  <collision>
+    <geometry>
+      <sphere radius="0.010"/>
     </geometry>
   </collision>
 </link>
 <joint name="BC_LEFT_J" type="fixed">
-  <origin xyz="0.20 -0.1 -0.0200"/>
+  <origin xyz="0.20 -0.1 -0.0030"/>
   <parent link="ebot_base"/>
   <child link="BC_LEFT"/>
@@ -222,16 +222,16 @@
   <visual>
     <geometry>
-      <sphere radius="0.015"/>
-    </geometry>
-    <material name="wheel_black"/>
-  </visual>
-  <collision>
-    <geometry>
-      <sphere radius="0.015"/>
+      <sphere radius="0.010"/>
+    </geometry>
+    <material name="wheel_black"/>
+  </visual>
+  <collision>
+    <geometry>
+      <sphere radius="0.010"/>
     </geometry>
   </collision>
 </link>
 <joint name="BC_RIGHT_J" type="fixed">
-  <origin xyz="-0.19 -0.1 -0.0200"/>
+  <origin xyz="-0.19 -0.1 -0.0030"/>
   <parent link="ebot_base"/>
   <child link="BC_RIGHT"/>
@@ -261,5 +261,5 @@
         <cylinder length="0.04" radius="0.03"/>
       </geometry>
-            <material name="wheel_black">
+      <material name="wheel_black">
         <color rgba="0.02 0.02 0.02 1.0"/>
       </material>

File: ebot_description/models/ebot/ebot_ros2_control.xacro (robot description, xacro)
@@ -4,8 +4,8 @@
     <ros2_control name="EbotSystem" type="system">
     <hardware>
-        <plugin>moveo_hardware/MoveoSystem</plugin>
+        <!-- <plugin>moveo_hardware/MoveoSystem</plugin>
         <param name="port">/dev/ttyACM0</param>
-        <param name="baudrate">115200</param>
-        <!-- <plugin>gz_ros2_control/GazeboSimSystem</plugin> -->
+        <param name="baudrate">115200</param> -->
+        <plugin>gz_ros2_control/GazeboSimSystem</plugin>
         <!-- <plugin>mock_components/GenericSystem</plugin> -->
         <!-- <param name="initial_positions">0 0 0 0</param> -->
@@ -14,15 +14,15 @@
         <command_interface name="position"/>
         <state_interface name="position"/>
-        <!-- <state_interface name="velocity"/> -->
+        <state_interface name="velocity"/>
         </joint>
         <joint name="Joint_2">
         <command_interface name="position"/>
         <state_interface name="position"/>
-        <!-- <state_interface name="velocity"/> -->
+        <state_interface name="velocity"/>
         </joint>
         <joint name="Joint_3">
         <command_interface name="position"/>
         <state_interface name="position"/>
-        <!-- <state_interface name="velocity"/> -->
+        <state_interface name="velocity"/>
         </joint>
         <joint name="Joint_4">
@@ -34,7 +34,7 @@
         <command_interface name="position"/>
         <state_interface name="position"/>
-        <!-- <state_interface name="velocity"/>/ -->
+        <state_interface name="velocity"/>/
         </joint>
-        <!-- <joint name="Gripper_Servo_Gear_Joint">
+        <joint name="Gripper_Servo_Gear_Joint">
         <command_interface name="position"/>
         <state_interface name="position"/>
@@ -53,5 +53,5 @@
         <state_interface name="position"/>
         <state_interface name="velocity"/>
-        </joint> -->
+        </joint>
     </ros2_control>
   </xacro:macro>

Commit message: added pid controll to ardiuno

File: ebot_description/models/ebot/ebot_description.xacro (robot description, xacro)
@@ -48,7 +48,7 @@
     </visual>
     <collision>
-      <origin xyz="0 0 0.12"/>
-      <geometry>
-        <box size="0.585 0.50 0.25"/>
+      <origin xyz="0 0 0.07"/>
+      <geometry>
+        <box size="0.510 0.30 0.10"/>
       </geometry>
     </collision>
@@ -64,10 +64,10 @@
   <link name="FWR">
     <inertial>
-      <xacro:cylinder_inertia c_mass="${wheel_mass}" r="0.08" l="0.05"/>
+      <xacro:cylinder_inertia c_mass="${wheel_mass}" r="0.0625" l="0.03"/>
     </inertial>
     <visual>
       <origin rpy="1.5708 0 0"/>
       <geometry>
-        <cylinder length="0.05" radius="0.08"/>
+        <cylinder length="0.03" radius="0.0625"/>
       </geometry>
       <material name="wheel_black">
@@ -78,10 +78,10 @@
       <origin rpy="1.5708 0 0"/>
       <geometry>
-        <cylinder length="0.05" radius="0.08"/>
+        <cylinder length="0.03" radius="0.0625"/>
       </geometry>
     </collision>
   </link>
   <joint name="FWRJ" type="continuous">
-    <origin xyz="0 -0.20 0.045"/>
+    <origin xyz="0 -0.18 0.045"/>
     <parent link="ebot_base"/>
     <child link="FWR"/>
@@ -91,10 +91,10 @@
   <link name="FWL">
     <inertial>
-      <xacro:cylinder_inertia c_mass="${wheel_mass}" r="0.08" l="0.05"/>
+      <xacro:cylinder_inertia c_mass="${wheel_mass}" r="0.0625" l="0.03"/>
     </inertial>
     <visual>
       <origin rpy="1.5708 0 0"/>
       <geometry>
-        <cylinder length="0.05" radius="0.08"/>
+        <cylinder length="0.03" radius="0.0625"/>
       </geometry>
      <material name="wheel_black">
@@ -105,10 +105,10 @@
       <origin rpy="1.5708 0 0"/>
       <geometry>
-        <cylinder length="0.05" radius="0.08"/>
+        <cylinder length="0.03" radius="0.0625"/>
       </geometry>
     </collision>
   </link>
   <joint name="FWLJ" type="continuous">
-    <origin xyz="0 0.20 0.045"/>
+    <origin xyz="0 0.18 0.045"/>
     <parent link="ebot_base"/>
     <child link="FWL"/>
@@ -119,6 +119,6 @@
   <!-- ===================== -->
   <!-- ===================== -->
-<!-- BALL CASTERS (4-DIRECTION SUPPORT) -->
-<!-- ===================== -->
+  <!-- BALL CASTERS (4-DIRECTION SUPPORT) -->
+  <!-- ===================== -->
 <!-- FRONT ball caster -->
 <link name="BC_FRONT">

Commit message: added nav2 and slam config and updated kdl lib for moveo

File: ebot_description/models/ebot/ebot_description.xacro (robot description, xacro)
@@ -54,5 +54,5 @@
     </visual>
     <collision>
-      <origin xyz="0 0 0.12"/>
+      <origin xyz="0 0 0.07"/>
       <geometry>
         <box size="0.510 0.30 0.10"/>

File: ebot_description/models/ebot/ebot_ros2_control.xacro (robot description, xacro)
@@ -29,10 +29,10 @@
         <command_interface name="position"/>
         <state_interface name="position"/>
-        <!-- <state_interface name="velocity"/> -->
+        <state_interface name="velocity"/>
         </joint>
         <joint name="Joint_5">
         <command_interface name="position"/>
         <state_interface name="position"/>
-        <state_interface name="velocity"/>/
+        <state_interface name="velocity"/>
         </joint>
         <joint name="Gripper_Servo_Gear_Joint">

File: moveo_description/urdf/moveo_urdf.urdf.xacro (robot description, xacro)
@@ -24,5 +24,5 @@
             <origin xyz="0 0 .13" rpy="0 0 0" />
             <geometry>
-                <mesh filename="package://moveo_description/meshes/base_link_col.STL" />
+                <box size="0.20 0.24 0.13"/>
             </geometry>
         </collision>
