Commit message: aruco reching pipeline completed

File: ebot_description/models/ebot/ebot_description.xacro (robot description, xacro)
@@ -7,4 +7,6 @@
   <xacro:include filename="$(find moveo_description)/urdf/moveo_urdf.urdf.xacro"/>
   <xacro:include filename="$(find ebot_description)/models/ebot/ebot_ros2_control.xacro"/>
+  <xacro:arg name="use_hardware" default="false"/>
+  <xacro:arg name="use_gripper" default="true"/>
   <xacro:moveo_arm prefix="moveo_"/>
   <!-- ===================== -->
@@ -133,32 +135,4 @@
     <dynamics damping="0.1" friction="0.0"/>
   </joint>
-  <!-- ===================== -->
-  <!-- TRANSMISSIONS -->
-  <!-- ===================== -->
-<!--
-  <transmission name="FWR_trans">
-    <type>transmission_interface/SimpleTransmission</type>
-    <joint name="FWRJ">
-      <hardwareInterface>hardware_interface/VelocityJointInterface</hardwareInterface>
-    </joint>
-    <actuator name="FWR_motor">
-      <mechanicalReduction>1</mechanicalReduction>
-    </actuator>
-  </transmission>
-  <transmission name="FWL_trans">
-    <type>transmission_interface/SimpleTransmission</type>
-    <joint name="FWLJ">
-      <hardwareInterface>hardware_interface/VelocityJointInterface</hardwareInterface>
-    </joint>
-    <actuator name="FWL_motor">
-      <mechanicalReduction>1</mechanicalReduction>
-    </actuator>
-  </transmission> -->
-  <!-- ===================== -->
-  <!-- OMNI CASTERS (SWIVEL + ROLL) -->
-  <!-- ===================== -->
-  <!-- ===================== -->
-<!-- BALL CASTERS (4-DIRECTION SUPPORT) -->
-<!-- ===================== -->
 <!-- FRONT ball caster -->
 <link name="BC_FRONT">
@@ -286,5 +260,11 @@
     <child link="imu_link"/>
   </joint>
-<xacro:ebot_ros2_control/>
-<xacro:ebot_gazebo_ros2_control/>
+<!-- ROS2 CONTROL -->
+<xacro:ebot_ros2_control
+    use_hardware="$(arg use_hardware)"
+    use_gripper="$(arg use_gripper)"/>
+<!-- Gazebo only if simulation -->
+<xacro:if value="$(arg use_gazebo)">
+  <xacro:ebot_gazebo_ros2_control/>
+</xacro:if>
 </robot>

File: ebot_description/models/ebot/ebot_ros2_control.xacro (robot description, xacro)
@@ -1,57 +1,58 @@
 <?xml version="1.0"?>
 <robot xmlns:xacro="http://www.ros.org/wiki/xacro">
-  <xacro:macro name="ebot_ros2_control">
+  <xacro:arg name="use_hardware" default="false"/>
+  <xacro:arg name="use_gripper" default="true"/>
+  <xacro:macro name="ebot_ros2_control" params="use_hardware use_gripper">
     <ros2_control name="EbotSystem" type="system">
-    <hardware>
-        <!-- <plugin>moveo_hardware/MoveoSystem</plugin>
-        <param name="port">/dev/ttyACM0</param>
-        <param name="baudrate">115200</param> -->
-        <plugin>gz_ros2_control/GazeboSimSystem</plugin>
-        <!-- <plugin>mock_components/GenericSystem</plugin> -->
-        <!-- <param name="initial_positions">0 0 0 0</param> -->
-    </hardware>
-        <joint name="Joint_1">
-        <command_interface name="position"/>
-        <state_interface name="position"/>
-        <state_interface name="velocity"/>
+      <!-- 🔁 Hardware Selection -->
+      <hardware>
+        <xacro:if value="$(arg use_hardware)">
+          <plugin>moveo_hardware/MoveoSystem</plugin>
+          <param name="port">/dev/ttyACM0</param>
+          <param name="baudrate">115200</param>
+        </xacro:if>
+        <xacro:unless value="$(arg use_hardware)">
+          <plugin>gz_ros2_control/GazeboSimSystem</plugin>
+        </xacro:unless>
+      </hardware>
+      <!-- 🔧 Arm Joints -->
+      <xacro:macro name="arm_joint" params="name">
+        <joint name="${name}">
+          <command_interface name="position"/>
+          <state_interface name="position"/>
+          <!-- ❗ Velocity only in simulation
+          <xacro:unless value="$(arg use_hardware)">
+            <state_interface name="velocity"/>
+          </xacro:unless> -->
         </joint>
-        <joint name="Joint_2">
-        <command_interface name="position"/>
-        <state_interface name="position"/>
-        <state_interface name="velocity"/>
-        </joint>
-        <joint name="Joint_3">
-        <command_interface name="position"/>
-        <state_interface name="position"/>
-        <state_interface name="velocity"/>
-        </joint>
-        <joint name="Joint_4">
-        <command_interface name="position"/>
-        <state_interface name="position"/>
-        <state_interface name="velocity"/>
-        </joint>
-        <joint name="Joint_5">
-        <command_interface name="position"/>
-        <state_interface name="position"/>
-        <state_interface name="velocity"/>
-        </joint>
+      </xacro:macro>
+      <xacro:arm_joint name="Joint_1"/>
+      <xacro:arm_joint name="Joint_2"/>
+      <xacro:arm_joint name="Joint_3"/>
+      <xacro:arm_joint name="Joint_4"/>
+      <xacro:arm_joint name="Joint_5"/>
+      <!-- 🤏 Gripper (optional) -->
+      <xacro:if value="$(arg use_gripper)">
         <joint name="Gripper_Servo_Gear_Joint">
-        <command_interface name="position"/>
-        <state_interface name="position"/>
+          <command_interface name="position"/>
+          <state_interface name="position"/>
         </joint>
         <joint name="Gripper_Idol_Gear_Joint">
-        <command_interface name="position"/>
-        <state_interface name="position"/>
+          <command_interface name="position"/>
+          <state_interface name="position"/>
         </joint>
-        <joint name="FWRJ">
+      </xacro:if>
+     <xacro:unless value="${use_hardware}">
+      <joint name="FWRJ">
         <command_interface name="velocity"/>
         <state_interface name="position"/>
         <state_interface name="velocity"/>
-        </joint>
-        <joint name="FWLJ">
+      </joint>
+      <joint name="FWLJ">
         <command_interface name="velocity"/>
         <state_interface name="position"/>
         <state_interface name="velocity"/>
-        </joint>
+      </joint>
+    </xacro:unless>
     </ros2_control>
   </xacro:macro>

File: moveo_description/urdf/sensors/intel_rgbd_cam_d435.urdf.xacro (robot description, xacro)
@@ -59,5 +59,5 @@
       <parent link="Link_5"/>
       <child link="camera_head_link" />
-      <origin xyz="0 0.01 0.50" rpy="0.0 ${camera_tilt_angle_deg * M_PI / 180} ${M_PI/2}"/>
+      <origin xyz="0 0.01 0.15" rpy="0.0 ${camera_tilt_angle_deg * M_PI / 180} ${M_PI/2}"/>
     </joint>
     <link name="camera_head_link">
@@ -141,5 +141,5 @@
           <clip>
             <near>0.05</near>
-            <far>1.5</far>
+            <far>4.5</far>
           </clip>
         </camera>

Commit message: boot strat loaded with and without arm

File: ebot_description/models/ebot/ebot_description.xacro (robot description, xacro)
@@ -2,4 +2,10 @@
 <robot name="ebot" xmlns:xacro="http://www.ros.org/wiki/xacro">
   <xacro:include filename="$(find ebot_description)/models/ebot/ebot.gazebo" />
+  <xacro:include filename="$(find ebot_description)/models/ebot/ebot_gazebo_control.xacro"/>
+  <xacro:include filename="$(find moveo_description)/urdf/moveo_urdf.urdf.xacro"/>
+  <xacro:include filename="$(find ebot_description)/models/ebot/ebot_ros2_control.xacro"/>
+  <xacro:arg name="use_hardware" default="false"/>
+  <xacro:arg name="use_gripper" default="true"/>
+  <xacro:arg name="use_arm" default="true"/>
   <!-- ===================== -->
   <!-- PROPERTIES -->
@@ -58,4 +64,15 @@
     <child link="ebot_base"/>
   </joint>
+  <!-- ===================== -->
+  <!-- ARM MOUNT -->
+  <!-- ===================== -->
+  <xacro:if value="$(arg use_arm)">
+    <xacro:moveo_arm prefix="moveo_"/>
+    <joint name="arm_mount_joint" type="fixed">
+      <parent link="ebot_base"/>
+      <child link="moveo_base_link"/>
+      <origin xyz="0 0 0.0" rpy="0 0 -1.5708"/>
+    </joint>
+  </xacro:if>
   <!-- ===================== -->
   <!-- DRIVE WHEELS -->
@@ -296,3 +313,13 @@
     <child link="camera"/>
   </joint>
+<!-- ROS2 CONTROL -->
+<xacro:if value="$(arg use_arm)">
+  <xacro:ebot_ros2_control
+      use_hardware="$(arg use_hardware)"
+      use_gripper="$(arg use_gripper)"/>
+</xacro:if>
+<!-- Gazebo only if simulation -->
+<xacro:if value="$(arg use_gazebo)">
+  <xacro:ebot_gazebo_ros2_control/>
+</xacro:if>
 </robot>

Commit message: dayafter

File: ebot_description/models/ebot/ebot_description.xacro (robot description, xacro)
@@ -99,5 +99,5 @@
     </collision>
   </link>
-  <joint name="FWRJ" type="continuous">
+  <joint name="FWRJ" type="fixed">
     <origin xyz="0 -0.18 0.045"/>
     <parent link="ebot_base"/>
@@ -126,5 +126,5 @@
     </collision>
   </link>
-  <joint name="FWLJ" type="continuous">
+  <joint name="FWLJ" type="fixed">
     <origin xyz="0 0.18 0.045"/>
     <parent link="ebot_base"/>
@@ -245,5 +245,6 @@
   </link>
   <joint name="lidar_joint" type="fixed">
-    <origin xyz="0.14 0.055 0.31"/>
+    <!-- <origin xyz="0.14 0.055 0.31"/> -->
+    <origin xyz="0.0 0.0 0.14"/>
     <parent link="ebot_base"/>
     <child link="laser"/>
@@ -297,7 +298,6 @@
     <child link="imu_link"/>
   </joint>
-  <link name="camera">
-    <visual>
-     <origin rpy="0 1.5708 0"/>
+  <!-- <link name="camera">
+    <visual>
       <geometry>
         <cylinder length="0.04" radius="0.01"/>
@@ -309,8 +309,8 @@
   </link>
   <joint name="camera_joint" type="fixed">
-    <origin xyz="0.14 0.052 0.24"/>
+    <origin xyz="0.14 0.052 0.24" rpy="1.57 3.14 1.57"/>
     <parent link="ebot_base"/>
     <child link="camera"/>
-  </joint>
+  </joint> -->
 <!-- ROS2 CONTROL -->
 <xacro:if value="$(arg use_arm)">

File: moveo_description/urdf/moveo_urdf.urdf.xacro (robot description, xacro)
@@ -346,5 +346,22 @@
         <mimic joint="Gripper_Idol_Gear_Joint" multiplier="1" offset="0" />
     </joint>
+    <link name="camera">
+        <visual>
+            <geometry>
+            <cylinder length="0.04" radius="0.01"/>
+            </geometry>
+            <material name="wheel_black">
+            <color rgba="0.02 0.02 0.02 1.0"/>
+            </material>
+        </visual>
+    </link>
+    <joint name="camera_joint" type="fixed">
+        <!-- slightly forward + slightly up -->
+        <origin xyz="0.02 -0.02 0.0" rpy="0 0 0"/>
+        <!-- IMPORTANT: attach to wrist, not base -->
+        <parent link="Gripper_Servo_Gear"/>
+        <child link="camera"/>
+    </joint>
 </xacro:macro>
-<xacro:include filename="sensors/intel_rgbd_cam_d435.urdf.xacro" />
+<!-- <xacro:include filename="sensors/intel_rgbd_cam_d435.urdf.xacro" /> -->
 </robot>
