Commit message: full body manipulation done

File: ebot_description/models/ebot/ebot_description.xacro (robot description, xacro)
@@ -241,5 +241,5 @@
   </link>
   <joint name="lidar_joint" type="fixed">
-    <origin xyz="0.2055 0 0.15"/>
+    <origin xyz="0.0 0 0.15"/>
     <parent link="ebot_base"/>
     <child link="laser"/>

File: moveo_description/urdf/moveo_urdf.urdf.xacro (robot description, xacro)
@@ -14,7 +14,7 @@
     <link name="${prefix}base_link">
         <visual>
-            <origin xyz="0 0.0 0.08" rpy="0 0 0" />
-            <geometry>
-                <box size="0.20 0.24 0.13"/>
+            <origin xyz="0.0 0.0 0.20" rpy="0 0 0" />
+            <geometry>
+                <box size="0.3 0.3 0.01"/>
                 <!-- <mesh filename="package://moveo_description/meshes/base_link.STL" /> -->
             </geometry>
@@ -26,5 +26,5 @@
             <origin xyz="0 0 .13" rpy="0 0 0" />
             <geometry>
-                <box size="0.20 0.24 0.13"/>
+                <box size="0.3 0.3 0.01"/>
             </geometry>
         </collision>
@@ -35,5 +35,5 @@
     </link>
     <joint name="Joint_1" type="revolute">
-	<origin xyz="0 0 .13" rpy="0 0 0" />
+	<origin xyz="0 0 .26" rpy="0 0 0" />
         <axis xyz="0 0 1" />
         <limit lower="-1.5707963268" upper="1.5707963268" effort="100" velocity="1.919862177191" />
@@ -174,4 +174,17 @@
         <limit lower="-1.5707963268" upper="1.5707963268" effort="100" velocity="1.919862177191" />
     </joint>
+    <link name="tool0">
+        <visual>
+            <geometry>
+                <sphere radius="0.001"/>
+            </geometry>
+        </visual>
+    </link>
+    <joint name="tool0_joint" type="fixed">
+        <parent link="Link_5"/>
+        <child link="tool0"/>
+        <!-- tune this -->
+        <origin xyz="0 0 0.14" rpy="0 0 0"/>
+    </joint>
     <link name="Gripper_Servo_Gear">
         <visual>
@@ -346,5 +359,22 @@
         <mimic joint="Gripper_Idol_Gear_Joint" multiplier="1" offset="0" />
     </joint>
+    <link name="camera">
+        <visual>
+            <geometry>
+            <cylinder length="0.04" radius="0.01"/>
+            </geometry>
+            <material name="wheel_black">
+            <color rgba="0.02 0.02 0.02 1.0"/>
+            </material>
+        </visual>
+    </link>
+    <joint name="camera_joint" type="fixed">
+        <!-- slightly forward + slightly up -->
+        <origin xyz="0.02 -0.02 0.0" rpy="0 0 0"/>
+        <!-- IMPORTANT: attach to wrist, not base -->
+        <parent link="Gripper_Servo_Gear"/>
+        <child link="camera"/>
+    </joint>
 </xacro:macro>
-<xacro:include filename="sensors/intel_rgbd_cam_d435.urdf.xacro" />
+<!-- <xacro:include filename="sensors/intel_rgbd_cam_d435.urdf.xacro" /> -->
 </robot>

Commit message: updated base bot visual

File: ebot_description/models/ebot/ebot_description.xacro (robot description, xacro)
@@ -47,10 +47,11 @@
     </inertial>
     <visual>
-      <origin xyz="0 0 0.07"/>
-      <geometry>
-        <box size="0.510 0.30 0.10"/>
-      </geometry>
-      <material name="gray">
-        <color rgba="0.5 0.5 0.5 0.8"/>
+      <origin xyz="0 0 0.02" rpy="0 0 1.5708"/>
+      <geometry>
+        <mesh filename="file:///home/rajvardhan/mobile_manipulator/install/ebot_description/share/ebot_description/meshes/Denis.stl"
+      scale="0.9 0.9 0.9"/>
+      </geometry>
+      <material name="carbon">
+        <color rgba="0.12 0.12 0.12 1.0"/>
       </material>
     </visual>
@@ -85,8 +86,17 @@
       <origin rpy="1.5708 0 0"/>
       <geometry>
-        <cylinder length="0.05" radius="0.0625"/>
-      </geometry>
-      <material name="wheel_black">
-        <color rgba="0.02 0.02 0.02 1.0"/>
+        <cylinder length="0.05" radius="0.05"/>
+      </geometry>
+      <material name="wheel_inner_white">
+        <color rgba="0.75294 0.75294 0.75294 1.0"/>
+      </material>
+    </visual>
+    <visual>
+      <origin rpy="1.5708 0 0"/>
+      <geometry>
+        <cylinder length="0.049" radius="0.0625"/>
+      </geometry>
+      <material name="wheel_green">
+        <color rgba="1 73 20 1"/>
       </material>
     </visual>
@@ -114,8 +124,17 @@
       <origin rpy="1.5708 0 0"/>
       <geometry>
-        <cylinder length="0.05" radius="0.0625"/>
-      </geometry>
-     <material name="wheel_black">
-        <color rgba="0.02 0.02 0.02 1.0"/>
+        <cylinder length="0.05" radius="0.05"/>
+      </geometry>
+      <material name="wheel_inner_white">
+        <color rgba="0.75294 0.75294 0.75294 1.0"/>
+      </material>
+    </visual>
+    <visual>
+      <origin rpy="1.5708 0 0"/>
+      <geometry>
+        <cylinder length="0.049" radius="0.0625"/>
+      </geometry>
+      <material name="wheel_green">
+        <color rgba="1 73 20 1"/>
       </material>
     </visual>

File: moveo_description/urdf/moveo_urdf.urdf.xacro (robot description, xacro)
@@ -23,4 +23,14 @@
             </material>
         </visual>
+        <visual>
+            <origin xyz="0.0 0.0 0.20" rpy="0 0 0" />
+            <geometry>
+                <!-- <box size="0.3 0.3 0.01"/> -->
+                <mesh filename="package://moveo_description/meshes/base_link.stl" />
+            </geometry>
+            <material name="">
+                <color rgba="0.75294 0.75294 0.75294 1" />
+            </material>
+        </visual>
         <collision>
             <origin xyz="0 0 .13" rpy="0 0 0" />
@@ -47,6 +57,6 @@
 		<mesh filename="package://moveo_description/meshes/Link_1_edited.STL" />
             </geometry>
-            <material name="">
-                <color rgba="0.75294 0.75294 0.75294 1" />
+            <material name="moveo_orange">
+                <color rgba="0.97 0.32 0.0 1.0"/>
             </material>
         </visual>
@@ -96,6 +106,6 @@
 		<mesh filename="package://moveo_description/meshes/Link_3_edited.STL" />
             </geometry>
-            <material name="">
-                <color rgba="0.75294 0.75294 0.75294 1" />
+            <material name="moveo_orange">
+                <color rgba="0.97 0.32 0.0 1.0"/>
             </material>
         </visual>
@@ -152,6 +162,6 @@
 		<mesh filename="package://moveo_description/meshes/Link_5_edited.STL" />
             </geometry>
-            <material name="">
-                <color rgba="0.75294 0.75294 0.75294 1" />
+            <material name="moveo_orange">
+                <color rgba="0.97 0.32 0.0 1.0"/>
             </material>
         </visual>
