Commit message: moveit controller and rgbd camera added

File: moveo_description/urdf/moveo_urdf.urdf.xacro (robot description, xacro)
@@ -2,4 +2,6 @@
 <robot name="moveo_description"
        xmlns:xacro="http://www.ros.org/wiki/xacro">
+    <xacro:arg name="use_camera" default="true"/>
+    <xacro:arg name="use_gazebo" default="true"/>
 <xacro:macro name="moveo_arm" params="prefix">
   <!-- <link name="world"/> -->
@@ -198,5 +200,5 @@
         <child link="Gripper_Servo_Gear" />
         <axis xyz="0 1 0" />
-        <limit lower="0" upper="1.5707963268" effort="100" velocity="0.5" />
+        <limit lower="-10" upper="10.5707963268" effort="100" velocity="0.5" />
     </joint>
     <link name="Gripper_Idol_Gear">
@@ -226,5 +228,5 @@
         <child link="Gripper_Idol_Gear" />
         <axis xyz="0 1 0" />
-        <limit lower="-1.5707963268" upper="0" effort="100" velocity="0.5" />
+        <limit lower="-10.5707963268" upper="10" effort="100" velocity="0.5" />
     </joint>
     <link name="Tip_Gripper_Idol">
@@ -275,5 +277,5 @@
         <child link="Tip_Gripper_Servo" />
         <axis xyz="0 1 0" />
-        <limit lower="0" upper="1.3" effort="100" velocity="0.5" />
+        <limit lower="-10" upper="10.3" effort="100" velocity="0.5" />
         <mimic joint="Gripper_Servo_Gear_Joint" multiplier="1" offset="0" />
     </joint>
@@ -283,5 +285,5 @@
         <child link="Tip_Gripper_Idol" />
         <axis xyz="0 1 0" />
-        <limit lower="3.14" upper="-3.14" effort="100" velocity="0.5" />
+        <limit lower="-13.14" upper="13.14" effort="100" velocity="0.5" />
         <mimic joint="Gripper_Idol_Gear_Joint" multiplier="-1" offset="0" />
     </joint>
@@ -312,5 +314,5 @@
         <child link="Pivot_Arm_Gripper_Servo" />
         <axis xyz="0 1 0" />
-        <limit lower="-1.5707963268" upper="1.5707963268" effort="100" velocity="0.5" />
+        <limit lower="-10.5707963268" upper="10.5707963268" effort="100" velocity="0.5" />
         <mimic joint="Gripper_Servo_Gear_Joint" multiplier="1" offset="0" />
     </joint>
@@ -341,7 +343,8 @@
         <child link="Pivot_Arm_Gripper_Idol" />
         <axis xyz="0 1 0" />
-        <limit lower="-1.5707963268" upper="1.5707963268" effort="100" velocity="0.5" />
+        <limit lower="-10.5707963268" upper="10.5707963268" effort="100" velocity="0.5" />
         <mimic joint="Gripper_Idol_Gear_Joint" multiplier="1" offset="0" />
     </joint>
 </xacro:macro>
+<xacro:include filename="sensors/intel_rgbd_cam_d435.urdf.xacro" />
 </robot>
